File: hardware/kicad/pico-serial-line.kicad_sch (KiCad schematic)
At the start: 99 parts, among them J1 USB_C, J2 RJ11, Q1 MMBTA42, Q2 MMBTA92, Q3 MMBTA42, Q4 MMBTA06, Q5 MMBTA06, SW1 BOOTSEL, SW2 RESET, U1 RP2040, U2 W25Q128JVS, U3 AP2112K-3.3, U4 USBLC6-2SC6, U5 Si3056-D-FS, U6 Si3018-F-FS, Y1 12MHz

Commit message: Line stick: line-voltage net class; the finisher keeps out of rule areas
The finishing router ignored rule areas: on the Line board it ran tracks
through the isolation gap and a screw's keep-out. It now treats every
no-track / no-via rule area as blocked (the hood and W boards had none of
their tracks there).

TIP, RING and the bridge's + (now LINE_*) keep 0.4 mm clearance; the
Si3018's low-voltage side (LS_*) gets 0.25 mm, so the line side can route.

Co-Authored-By: Claude Opus 5.5 <noreply@anthropic.com>
Claude-Session: https://claude.ai/code/session_013PRsUCpxazyipPn5UGGkF8
Connections:
- net LS_RING_F renamed LINE_RING_F
- net LS_RING_M renamed LINE_RING_M
- net LS_TIP_F renamed LINE_TIP_F
- net LS_TIP_M renamed LINE_TIP_M
- net LS_TIP_P renamed LINE_TIP_P
- net LS_VP renamed LINE_VP
Other:
- moved on the sheet: C29, D4, F2, FB1, FB2, Q1, R27, R28, RV1

Commit message: schematic: wb variant (TLV320AIC3204, PE-65848 footprint and symbol)
Co-Authored-By: Claude Opus 5.5 <noreply@anthropic.com>
Claude-Session: https://claude.ai/code/session_013PRsUCpxazyipPn5UGGkF8
Other:
- note added: "Status LEDs"
- note removed: "Status LEDs (optional, not fitted)"
Changed lines of the file:
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@@
 		(effects (font (size 2 2) (bold yes)) (justify left bottom))
 	)
-	(text "Status LEDs (optional, not fitted)"
+	(text "Status LEDs"
 		(exclude_from_sim no)
 		(at 345.44 21.59 0)
