File: hardware/kicad/pico-serial-w.kicad_pcb (KiCad board)
At the start: 4 copper layers, 50.6 x 55.3 mm, 88 parts, among them J1 USB_C, J2 DB25_Female, SW1 BOOTSEL, SW2 RESET, SW3 PAIR, U1 RP2040, U2 W25Q128JVS, U3 AP2112K-3.3, U4 USBLC6-2SC6, U5 SP3238EEA, U6 MAX3243EIDBR, U7 RM2, Y1 12MHz

Commit message: Point repository references at the D-Modem organisation
The repositories moved from Neo-Desktop to the D-Modem GitHub
organisation: D-Modem-RE is now D-Modem/D-Modem, pico-serial is
D-Modem/hardware, modemmenu (PBX-Modem) is D-Modem/menu, bbs-sec is
D-Modem/bbs and go3270-sec is D-Modem/go3270.  Update links, module
paths, submodule URLs and source-location strings to match.  Copyright
notices still name Neo-Desktop.

Co-Authored-By: Claude Opus 5.5 <noreply@anthropic.com>
Claude-Session: https://claude.ai/code/session_01B82eRUwD2JJ5d6fgHmpVTw
Other:
- board text added: "github.com/D-Modem/hardware"
- board text removed: "github.com/Neo-Desktop/pico-serial"
Changed lines of the file:
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@@
 		)
 	)
-	(gr_text "github.com/Neo-Desktop/pico-serial"
+	(gr_text "github.com/D-Modem/hardware"
 		(at 0 4.45 0)
 		(layer "B.SilkS")
