File: hardware/kicad/pico-serial.kicad_pcb (KiCad board)
At the start: 4 copper layers, 37 x 38 mm, 81 parts, among them J1 USB_C, J2 DB25_Female, SW1 BOOTSEL, SW2 RESET, U1 RP2040, U2 W25Q128JVS, U3 AP2112K-3.3, U4 USBLC6-2SC6, U5 SP3238EEA, U6 MAX3243EIDBR, Y1 12MHz

Commit message: Hardware: route the PCB; DRC clean, matches the schematic
- Routed with Freerouting 1.9 (rounds, each from the last) plus a small
  A* grid router in build_pcb.py for what it leaves; deterministic, and
  it tries a few pass counts if one leaves anything.
- In1.Cu solid GND; In2.Cu signals then a +3V3 pour; GND pours top and
  bottom. Every GND/+3V3 pad has its own via (U1's +3V3 inward, under
  the package); USB-C D+/D- corridor kept clear of vias.
- Net names come from KiCad's own export of the schematic, so DRC's
  schematic parity check passes; DNP/BOM flags match the symbols.
- Edge keep-out band (Freerouting ignores KiCad's edge clearance) and
  keep-outs around the USB-C's plastic pegs.
- Placement tweaks for routability; test pads moved behind the flash;
  licence and Source Location on the silkscreen.
- kicad-cli DRC (KiCad 9.0.9, 9.0 libraries): 0 violations, 0
  unconnected, 0 parity issues. ERC: 0.

Co-Authored-By: Claude Opus 5.5 <noreply@anthropic.com>
Claude-Session: https://claude.ai/code/session_013PRsUCpxazyipPn5UGGkF8
Parts:
- moved TP8 22.0 mm to (-9.50, 23.8)
- moved TP10 12.4 mm to (6.50, 26.2)
- moved TP5 12.4 mm to (6.50, 23.6)
- moved R5 4.25 mm to (-11.0, 20.1)
- moved TP6 4.00 mm to (9.10, 23.6)
- moved TP7 4.00 mm to (11.7, 23.6)
- moved TP11 4.00 mm to (9.10, 26.2)
- moved TP12 4.00 mm to (11.7, 26.2)
- moved C10 3.94 mm to (0.40, 21.6), turned to 0 degrees
- moved R4 3.81 mm to (-11.0, 19.0)
- moved TP9 3.44 mm to (14.3, 23.6)
- moved TP1 3.44 mm to (6.50, 21.0)
- moved TP2 3.44 mm to (9.10, 21.0)
- moved TP3 3.44 mm to (11.7, 21.0)
- moved TP4 3.44 mm to (14.3, 21.0)
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Connections:
- net A_CTS renamed /A_CTS
- net A_DCD renamed /A_DCD
- net A_DSR renamed /A_DSR
- net A_DTR renamed /A_DTR
- net A_R1OUTB renamed /A_R1OUTB
- net A_RI renamed /A_RI
- net A_RTS renamed /A_RTS
- net A_RX renamed /A_RX
- net A_SHDN_N renamed /A_SHDN_N
- net A_STATUS renamed /A_STATUS
- net A_TX renamed /A_TX
- net BOOTSEL_SW renamed /BOOTSEL_SW
- net B_CTS renamed /B_CTS
- net B_DCD renamed /B_DCD
- net B_DSR renamed /B_DSR
- net B_DTR renamed /B_DTR
- net B_FORCEOFF_N renamed /B_FORCEOFF_N
- net B_INVALID renamed /B_INVALID
- net B_RI renamed /B_RI
- net B_RTS renamed /B_RTS
- net B_RX renamed /B_RX
- net B_TX renamed /B_TX
- net CC1 renamed /CC1
- net CC2 renamed /CC2
- net CPA_C1M renamed /CPA_C1M
- net CPA_C1P renamed /CPA_C1P
- net CPA_C2M renamed /CPA_C2M
- net CPA_C2P renamed /CPA_C2P
- net CPA_VM renamed /CPA_VM
- net CPA_VP renamed /CPA_VP
- net CPB_C1M renamed /CPB_C1M
- net CPB_C1P renamed /CPB_C1P
- net CPB_C2M renamed /CPB_C2M
- net CPB_C2P renamed /CPB_C2P
- net CPB_VM renamed /CPB_VM
- net CPB_VP renamed /CPB_VP
- net DB25_FG renamed /DB25_FG
- net GP28 renamed /GP28
- net LED_CD renamed /LED_CD
- net LED_CD_A renamed /LED_CD_A
- net LED_PWR renamed /LED_PWR
- net LED_PWR_A renamed /LED_PWR_A
- net LED_RD renamed /LED_RD
- net LED_RD_A renamed /LED_RD_A
- net LED_RI renamed /LED_RI
- net LED_RI_A renamed /LED_RI_A
- net LED_SD renamed /LED_SD
- net LED_SD_A renamed /LED_SD_A
- net LED_TR renamed /LED_TR
- net LED_TR_A renamed /LED_TR_A
- net QSPI_SCLK renamed /QSPI_SCLK
- net QSPI_SD0 renamed /QSPI_SD0
- net QSPI_SD1 renamed /QSPI_SD1
- net QSPI_SD2 renamed /QSPI_SD2
- net QSPI_SD3 renamed /QSPI_SD3
- net QSPI_SS renamed /QSPI_SS
- net RS_CTS renamed /RS_CTS
- net RS_DCD renamed /RS_DCD
- net RS_DSR renamed /RS_DSR
- net RS_DTR renamed /RS_DTR
- net RS_FORCEON renamed /RS_FORCEON
- net RS_RI renamed /RS_RI
- net RS_RTS renamed /RS_RTS
- net RS_RXD renamed /RS_RXD
- net RS_TXD renamed /RS_TXD
- net RUN renamed /RUN
- net SWCLK renamed /SWCLK
- net SWDIO renamed /SWDIO
- net USB_CONN_DM renamed /USB_CONN_DM
- net USB_CONN_DP renamed /USB_CONN_DP
- net USB_DM renamed /USB_DM
- net USB_DP renamed /USB_DP
- net USB_SHIELD renamed /USB_SHIELD
- net VBUS_IN renamed /VBUS_IN
- net VBUS_SENSE renamed /VBUS_SENSE
- net XIN renamed /XIN
- net XOUT renamed /XOUT
- net XTAL_OUT renamed /XTAL_OUT
- J1 pad A8: (no net) -> unconnected-(J1-SBU1-PadA8)
- J1 pad B8: (no net) -> unconnected-(J1-SBU2-PadB8)
- J2 pad 10: (no net) -> unconnected-(J2-Pad10)
- J2 pad 11: (no net) -> unconnected-(J2-Pad11)
- J2 pad 12: (no net) -> unconnected-(J2-Pad12)
- J2 pad 13: (no net) -> unconnected-(J2-Pad13)
- J2 pad 14: (no net) -> unconnected-(J2-P14-Pad14)
- J2 pad 15: (no net) -> unconnected-(J2-P15-Pad15)
- J2 pad 16: (no net) -> unconnected-(J2-P16-Pad16)
- J2 pad 17: (no net) -> unconnected-(J2-P17-Pad17)
- J2 pad 18: (no net) -> unconnected-(J2-P18-Pad18)
- J2 pad 19: (no net) -> unconnected-(J2-P19-Pad19)
- J2 pad 21: (no net) -> unconnected-(J2-P21-Pad21)
- J2 pad 23: (no net) -> unconnected-(J2-P23-Pad23)
- J2 pad 24: (no net) -> unconnected-(J2-P24-Pad24)
- J2 pad 25: (no net) -> unconnected-(J2-P25-Pad25)
- J2 pad 9: (no net) -> unconnected-(J2-Pad9)
- U3 pad 4: (no net) -> unconnected-(U3-NC-Pad4)
- U6 pad 20: (no net) -> unconnected-(U6-ROUT2B-Pad20)
Routing:
- net +3V3: track 21.3 -> 99.4 mm, vias 21 -> 30
- net +1V1: track 0.00 -> 75.2 mm, vias 0 -> 6
- net /A_R1OUTB: track 0.00 -> 56.8 mm, vias 0 -> 2
- net /RS_FORCEON: track 0.00 -> 50.2 mm, vias 0 -> 2
- net /B_TX: track 0.00 -> 41.0 mm, vias 0 -> 2
- net /RUN: track 0.00 -> 39.6 mm, vias 0 -> 3
- net /RS_TXD: track 0.00 -> 39.1 mm, vias 0 -> 2
- net /SWCLK: track 0.00 -> 39.0 mm, vias 0 -> 2
- net /SWDIO: track 0.00 -> 39.0 mm, vias 0 -> 1
- net /A_STATUS: track 0.00 -> 38.3 mm, vias 0 -> 2
- net VBUS: track 0.00 -> 35.4 mm, vias 0 -> 2
- net /B_RX: track 0.00 -> 34.8 mm, vias 0 -> 4
- net /RS_RTS: track 0.00 -> 33.9 mm, vias 0 -> 2
- net /RS_CTS: track 0.00 -> 32.7 mm, vias 0 -> 2
- net /RS_DCD: track 0.00 -> 31.2 mm, vias 0 -> 2
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
Commit message: hardware: lay out and route the 4-layer PCB
build_pcb.py builds the board from the schematic: outline, JLC rules,
net classes, placement on both sides, GND/+3V3 fanout, Freerouting 1.9
plus a rip-up finisher, then pours. DRC, ERC and schematic parity are
clean. Adds Gerbers, drill and JLC placement files, renders, docs, and a
CI workflow that checks ERC, DRC and parity.

Co-Authored-By: Claude Opus 5.5 <noreply@anthropic.com>
Claude-Session: https://claude.ai/code/session_013PRsUCpxazyipPn5UGGkF8
Parts:
- moved R12 25.6 mm to (-9.00, 15.4), turned to 0 degrees
- moved R13 25.6 mm to (15.0, 6.60), turned to 90 degrees
- moved C23 18.6 mm to (-13.2, 15.4)
- moved C24 18.6 mm to (-11.0, 15.4)
- moved C29 18.6 mm to (5.40, 15.4)
- moved C30 18.6 mm to (7.60, 15.4)
- moved C21 18.5 mm to (-16.9, 11.4), turned to 180 degrees
- moved C27 18.5 mm to (1.60, 11.4), turned to 180 degrees
- moved C19 18.5 mm to (-16.9, 9.70), turned to 180 degrees
- moved C25 18.5 mm to (1.60, 9.70), turned to 180 degrees
- moved C22 18.5 mm to (-16.9, 7.95), turned to 180 degrees
- moved C28 18.5 mm to (1.60, 7.95), turned to 180 degrees
- moved C20 18.5 mm to (-16.9, 6.20), turned to 180 degrees
- moved C26 18.5 mm to (1.60, 6.20), turned to 180 degrees
- moved U5 18.5 mm to (-10.0, 9.60)
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Routing:
- net /A_R1OUTB: track 56.8 -> 6.52 mm, vias 2 -> 1
- net /B_RTS: track 12.5 -> 61.5 mm, vias 1 -> 5
- net /A_RX: track 27.6 -> 67.8 mm, vias 2 -> 3
- net /B_INVALID: track 7.96 -> 46.0 mm
- net /A_STATUS: track 38.3 -> 8.82 mm, vias 2 -> 1
- net /B_FORCEOFF_N: track 11.9 -> 38.0 mm, vias 1 -> 2
- net /A_TX: track 21.6 -> 44.9 mm, vias 1 -> 3
- net /A_CTS: track 16.1 -> 39.1 mm
- net /RS_FORCEON: track 50.2 -> 34.1 mm, vias 2 -> 1
- net /A_RTS: track 8.96 -> 24.6 mm
- net /A_DTR: track 12.3 -> 25.8 mm, vias 1 -> 2
- net /SWCLK: track 39.0 -> 50.0 mm, vias 2 -> 4
- net /B_DCD: track 13.8 -> 24.1 mm, vias 2 -> 3
- net /B_DTR: track 25.1 -> 15.6 mm, vias 3 -> 1
- net /RS_TXD: track 39.1 -> 29.9 mm
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
Commit message: Point repository references at the D-Modem organisation
The repositories moved from Neo-Desktop to the D-Modem GitHub
organisation: D-Modem-RE is now D-Modem/D-Modem, pico-serial is
D-Modem/hardware, modemmenu (PBX-Modem) is D-Modem/menu, bbs-sec is
D-Modem/bbs and go3270-sec is D-Modem/go3270.  Update links, module
paths, submodule URLs and source-location strings to match.  Copyright
notices still name Neo-Desktop.

Co-Authored-By: Claude Opus 5.5 <noreply@anthropic.com>
Claude-Session: https://claude.ai/code/session_01B82eRUwD2JJ5d6fgHmpVTw
Other:
- board text added: "github.com/D-Modem/hardware"
- board text removed: "github.com/Neo-Desktop/pico-serial"
Changed lines of the file:
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@@
 		)
 	)
-	(gr_text "github.com/Neo-Desktop/pico-serial"
+	(gr_text "github.com/D-Modem/hardware"
 		(at 0 4.45 0)
 		(layer "B.SilkS")
